File: KiCAD/fujiflex.kicad_pcb (KiCad board)
At the start: 2 copper layers, 27.7 x 30 mm, 35 parts, among them IC1 XC3S200A-4VQG100C, IC2 AT25SF041B-MAHD-T, J23 505278-1933, U1 AP2127N-1.2

Commit message: update
Parts:
- C1, C2: value C_Small -> 1uF
- renumbered J23 to J1, IC1 to U1, IC2 to U2, U1 to U3
