File: KiCAD/fujiflex.kicad_pcb (KiCad board)
At the start: 2 copper layers, 27.7 x 30 mm, 35 parts, among them J1 505278-1933, U1 XC3S200A-4VQG100C, U2 AT25SF041B-MAHD-T, U3 AP2127N-1.2

Commit message: moar stitching vias
Routing:
- net GND: vias 133 -> 135
Changed lines of the file:
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@@
+	)
+	(via
+		(at 157.132418 110.54439)
+		(size 0.35)
+		(drill 0.15)
+		(layers "F.Cu" "B.Cu")
+		(teardrops
+			(best_length_ratio 0.5)
+			(max_length 2)
+			(best_width_ratio 1)
+			(max_width 2)
+			(curve_points 7)
+			(filter_ratio 0.9)
+			(enabled yes)
+			(allow_two_segments yes)
+			(prefer_zone_connections yes)
+		)
+		(net 1)
 	)
 	(via
@@
 		(size 0.35)
 		(drill 0.15)
+		(layers "F.Cu" "B.Cu")
+		(teardrops
+			(best_length_ratio 0.5)
+			(max_length 2)
+			(best_width_ratio 1)
+			(max_width 2)
+			(curve_points 7)
+			(filter_ratio 0.9)
+			(enabled yes)
+			(allow_two_segments yes)
+			(prefer_zone_connections yes)
+		)
+		(net 1)
+	)
+	(via
+		(at 158.037198 110.188315)
+		(size 0.35)
+		(drill 0.15)
