File: KiCAD/fujiflex.kicad_sch (KiCad schematic)
At the start: 35 parts, among them IC1 XC3S200A-4VQG100C, IC2 AT25SF041B-MAHD-T, J23 505278-1933, U1 AP2127N-1.2

Commit message: update
Parts:
- C1, C2: value C_Small -> 1uF
- renumbered J23 to J1, IC1 to U1, IC2 to U2, U1 to U3
Changed lines of the file:
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@@
 			)
 		)
-		(property "Value" "C_Small"
+		(property "Value" "1uF"
 			(at 243.6241 38.0484 0)
 			(effects
@@
 		(on_board yes)
 		(dnp no)
-		(property "Reference" "IC1"
+		(property "Reference" "U1"
 			(at 104.0249 71.325 0)
 			(effects
@@
 			(project "fujiflex"
 				(path "/39897c5c-2595-480c-98d1-c9e79572b20a"
-					(reference "IC1")
+					(reference "U1")
 					(unit 1)
 				)
@@
 		(dnp no)
 		(fields_autoplaced yes)
-		(property "Reference" "U1"
+		(property "Reference" "U3"
 			(at 252.73 28.2405 0)
 			(effects
@@
 			(project "fujiflex"
 				(path "/39897c5c-2595-480c-98d1-c9e79572b20a"
-					(reference "U1")
+					(reference "U3")
 					(unit 1)
 				)
@@
 		(dnp no)
 		(fields_autoplaced yes)
-		(property "Reference" "IC2"
+		(property "Reference" "U2"
 			(at 212.09 125.4463 0)
 			(effects
@@
 			(project "fujiflex"
 				(path "/39897c5c-2595-480c-98d1-c9e79572b20a"
-					(reference "IC2")
+					(reference "U2")
 					(unit 1)
 				)
@@
 			)
 		)
-		(property "Value" "C_Small"
+		(property "Value" "1uF"
 			(at 265.2141 38.0484 0)
 			(effects
@@
 		(on_board yes)
 		(dnp no)
-		(property "Reference" "J23"
+		(property "Reference" "J1"
 			(at 210.82 51.7863 0)
 			(effects
@@
 			(project "fujiflex"
 				(path "/39897c5c-2595-480c-98d1-c9e79572b20a"
-					(reference "J23")
-					(unit 1)
-				)
+					(reference "J1")
+					(unit 1)
+				)

Commit message: fix schematic
Other:
- note removed: "x5 0.1uF"
- moved on the sheet: C10
Changed lines of the file:
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@@
 	)
 	(junction
-		(at 38.1 170.18)
-		(diameter 0)
-		(color 0 0 0 0)
-	)
-	(junction
 		(at 160.02 148.59)
 		(diameter 0)
@@
 	)
 	(junction
-		(at 38.1 162.56)
-		(diameter 0)
-		(color 0 0 0 0)
-	)
-	(junction
 		(at 33.02 147.32)
 		(diameter 0)
@@
 	(wire
 		(pts
-			(xy 43.18 170.18) (xy 38.1 170.18)
-		)
-		(stroke
-			(width 0)
-			(type default)
-		)
-	)
-	(wire
-		(pts
 			(xy 22.86 168.91) (xy 22.86 170.18)
 		)
@@
 	(wire
 		(pts
-			(xy 43.18 163.83) (xy 43.18 162.56)
+			(xy 38.1 163.83) (xy 38.1 162.56)
 		)
 		(stroke
@@
 	(wire
 		(pts
-			(xy 43.18 168.91) (xy 43.18 170.18)
+			(xy 38.1 168.91) (xy 38.1 170.18)
 		)
 		(stroke
@@
 	(wire
 		(pts
-			(xy 38.1 162.56) (xy 38.1 163.83)
-		)
-		(stroke
-			(width 0)
-			(type default)
-		)
-	)
-	(wire
-		(pts
 			(xy 27.94 170.18) (xy 30.48 170.18)
 		)
@@
 	(wire
 		(pts
-			(xy 38.1 168.91) (xy 38.1 170.18)
-		)
-		(stroke
-			(width 0)
-			(type default)
-		)
-	)
-	(wire
-		(pts
 			(xy 157.48 146.05) (xy 162.56 146.05)
 		)
@@
 	(wire
 		(pts
-			(xy 43.18 162.56) (xy 38.1 162.56)
-		)
-		(stroke
-			(width 0)
-			(type default)
-		)
-	)
-	(wire
-		(pts
 			(xy 234.95 137.16) (xy 242.57 137.16)
 		)
@@
 		)
 	)
-	(text "x5 0.1uF"
+	(text "x4 0.1uF"
 		(exclude_from_sim no)
-		(at 48.1452 169.3341 0)
+		(at 45.6052 169.3341 0)
 		(effects
 			(font
@@
 	(symbol
 		(lib_id "Device:C_Small")
-		(at 43.18 166.37 0)
+		(at 38.1 166.37 0)
 		(unit 1)
 		(exclude_from_sim no)
@@
 		(dnp no)
 		(property "Reference" "C10"
-			(at 43.6312 164.4331 0)
+			(at 38.5512 164.4331 0)
 			(effects
 				(font
@@
 		)
 		(property "Value" "0.1uF"
-			(at 44.2341 167.5884 0)
+			(at 39.1541 167.5884 0)
 			(effects
 				(font
@@
 		)
 		(property "Footprint" "Capacitor_SMD:C_0402_1005Metric"
-			(at 43.18 166.37 0)
+			(at 38.1 166.37 0)
 			(effects
 				(font
@@
 		)
 		(property "Datasheet" "~"
-			(at 43.18 166.37 0)
+			(at 38.1 166.37 0)
 			(effects
 				(font
@@
 		)
 		(property "Description" "Unpolarized capacitor, small symbol"
-			(at 43.18 166.37 0)
+			(at 38.1 166.37 0)
 			(effects
 				(font

Commit message: fix LDO blunder
Parts:
- U3: value AP2127N-1.2 -> TPS7A0512PDBZR
Changed lines of the file:
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@@
 			)
 		)
-		(property "Value" "AP2127N-1.2"
+		(property "Value" "TPS7A0512PDBZR"
 			(at 252.73 30.6648 0)
 			(effects
@@
 			)
 		)
-		(property "Datasheet" "https://www.diodes.com/assets/Datasheets/AP2127.pdf"
+		(property "Datasheet" ""
 			(at 252.73 34.29 0)
 			(effects
@@
 			)
 		)
-		(property "Description" "300mA low dropout linear regulator, shutdown pin, 2.5V-6V input voltage, 1.2V fixed positive output, SOT-23 package"
+		(property "Description" ""
 			(at 252.73 34.29 0)
 			(effects

Commit message: pcb fixes
- tie IR button pin high
- minor layout/routing tweaks
- silkscreen edits
- updated gerbers
Connections:
- net +3.3V: now also U1.70 (IO_L05P_1)
- no-connect marks 41 -> 40
Changed lines of the file:
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@@
 (kicad_sch
-	(version 20231120)
+	(version 20240101)
 	(generator "eeschema")
-	(generator_version "8.0")
+	(generator_version "8.99")
 	(paper "A4")
 	(junction
@@
 	)
 	(junction
+		(at 148.59 83.82)
+		(diameter 0)
+		(color 0 0 0 0)
+	)
+	(junction
 		(at 55.88 124.46)
 		(diameter 0)
@@
 	)
 	(no_connect
-		(at 140.97 83.82)
-	)
-	(no_connect
 		(at 80.01 40.64)
 	)
@@
 	(wire
 		(pts
-			(xy 148.59 33.02) (xy 148.59 88.9)
+			(xy 148.59 33.02) (xy 148.59 83.82)
 		)
 		(stroke
@@
 	(wire
 		(pts
+			(xy 140.97 83.82) (xy 148.59 83.82)
+		)
+		(stroke
+			(width 0)
+			(type default)
+		)
+	)
+	(wire
+		(pts
 			(xy 148.59 91.44) (xy 140.97 91.44)
 		)
@@
 		)
 		(stroke
+			(width 0)
+			(type default)
+		)
+	)
+	(wire
+		(pts
+			(xy 148.59 83.82) (xy 148.59 88.9)
+		)
+		(stroke
