File: KiCAD/fujiflex.kicad_sch (KiCad schematic)
At the start: 33 parts, among them J1 505278-1933, U1 XC3S200A-4VQG100C, U2 AT25SF041B-MAHD-T, U3 TPS7A0512PDBZR

Commit message: pcbway prod files
Parts:
- removed R4: 0, Resistor_SMD:R_0402_1005Metric, symbol Device:R_Small
- added TP1: TestPoint, SamacSys:TestPoint_Pad_D0.75mm, symbol Connector:TestPoint
- U2: renamed from U1; footprint QFP50P1600X1600X120-100N -> SamacSys:QFP50P1600X1600X120-100N
- U3: renamed from U2; footprint SON50P300X200X60-9N-D -> SamacSys:SON50P300X200X60-9N-D
- renumbered C9 to C10, C10 to C11, C11 to C12, C12 to C7, C7 to C8, C8 to C9, TP7 to TP10, TP8 to TP11, TP9 to TP12, TP3 to TP2, TP2 to TP3, TP1 to TP4, TP10 to TP6, TP11 to TP7, TP4 to TP8, TP6 to TP9, U3 to U1
Connections:
- net +3.3V: now also C7.1, R3.1, U3.3 (~{WP_(IO2})), U3.7 (~{HOLD_(IO3})), U3.8 (VCC); no longer U2.48 (IO_L10P_2/INIT_B)
- net at U2.100 (PROG_B): now also TP1.1
