File: KiCAD/6 Layer Compatible/fujiflex.kicad_sch (KiCad schematic)
At the start: 33 parts, among them J1 505278-1933, U1 XC3S200A-4VQG100C, U2 AT25SF041B-MAHD-T, U3 AP2127N-1.2

Commit message: minor layout updates
-updated grounding and some via sizes
-fixed IR button on 6L version
-updated gerbers
Parts:
- U3: value AP2127N-1.2 -> TPS7A0512PDBZR
Connections:
- net +3.3V: now also U1.70 (IO_L05P_1)
- no-connect marks 41 -> 40
Changed lines of the file:
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@@
 (kicad_sch
-	(version 20231120)
+	(version 20240101)
 	(generator "eeschema")
-	(generator_version "8.0")
+	(generator_version "8.99")
 	(paper "A4")
 	(junction
@@
 	)
 	(junction
+		(at 148.59 83.82)
+		(diameter 0)
+		(color 0 0 0 0)
+	)
+	(junction
 		(at 55.88 96.52)
 		(diameter 0)
@@
 	)
 	(no_connect
-		(at 140.97 83.82)
-	)
-	(no_connect
 		(at 80.01 40.64)
 	)
@@
 	(wire
 		(pts
-			(xy 148.59 33.02) (xy 148.59 88.9)
+			(xy 148.59 33.02) (xy 148.59 83.82)
 		)
 		(stroke
@@
 	(wire
 		(pts
+			(xy 148.59 83.82) (xy 148.59 88.9)
+		)
+		(stroke
+			(width 0)
+			(type default)
+		)
+	)
+	(wire
+		(pts
 			(xy 194.31 93.98) (xy 194.31 86.36)
 		)
@@
 	(wire
 		(pts
+			(xy 140.97 83.82) (xy 148.59 83.82)
+		)
+		(stroke
+			(width 0)
+			(type default)
+		)
+	)
+	(wire
+		(pts
 			(xy 87.63 24.13) (xy 90.17 24.13)
 		)
@@
 			)
 		)
-		(property "Value" "AP2127N-1.2"
+		(property "Value" "TPS7A0512PDBZR"
 			(at 252.73 30.6648 0)
 			(effects
