File: output_adapters/typeA/typeA.kicad_pcb (KiCad board)
At the start: 2 copper layers, 20.8 x 26.5 mm, 10 parts, among them J1 HC-HDMI0019T-1, J2 505278-1933, U1 ESD204DQAR-ES, U2 ESD204DQAR-ES, U3 ESD204DQAR-ES

Commit message: add dimensions
Other:
- board text added: "M2 screwhole x4"
Changed lines of the file:
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@@
 		(pad_to_mask_clearance 0)
 		(allow_soldermask_bridges_in_footprints no)
+		(grid_origin 170.25 105.5)
 		(pcbplotparams
 			(layerselection 0x00010f8_ffffffff)
@@
 		)
 	)
+	(gr_line
+		(start 167.5 88)
+		(end 170.25 90.5)
+		(stroke
+			(width 0.1)
+			(type default)
+		)
+		(layer "Cmts.User")
+	)
 	(gr_arc
 		(start 168.164203 89.121795)
@@
 		)
 	)
+	(gr_text "M2 screwhole x4"
+		(at 154.5 88 0)
+		(layer "Cmts.User")
+		(effects
+			(font
+				(size 1 1)
+				(thickness 0.15)
+			)
+			(justify left bottom)
+		)
+	)
+	(dimension
+		(type aligned)
+		(layer "Edge.Cuts")
+		(pts
+			(xy 170.25 105.5) (xy 181.75 105.5)
+		)
+		(height 3.25)
+		(gr_text "11.5000 mm"
+			(at 176 110.25 0)
+			(layer "Edge.Cuts")
+			(effects
+				(font
+					(size 1 1)
+					(thickness 0.15)
+				)
+			)
+		)
+		(format
+			(prefix "")
+			(suffix "")
+			(units 3)
+			(units_format 1)
+			(precision 4)
+		)
+		(style
+			(thickness 0.05)
+			(arrow_length 1.27)
+			(text_position_mode 2)
+			(extension_height 0.58642)
+			(extension_offset 0.5) keep_text_aligned)
+	)
+	(dimension
+		(type aligned)
+		(layer "Edge.Cuts")
+		(pts
+			(xy 169.15 90.5) (xy 171.35 90.5)
+		)
+		(height -4.25)
+		(gr_text "2.2000 mm"
+			(at 170.25 85.1 0)
+			(layer "Edge.Cuts")
+			(effects
+				(font
+					(size 1 1)
+					(thickness 0.15)
+				)
+			)
+		)
+		(format
+			(prefix "")
+			(suffix "")
+			(units 3)
+			(units_format 1)
+			(precision 4)
+		)
+		(style
+			(thickness 0.05)
+			(arrow_length 1.27)
+			(text_position_mode 0)
+			(extension_height 0.58642)
+			(extension_offset 0.5) keep_text_aligned)
+	)
+	(dimension
+		(type aligned)
+		(layer "Edge.Cuts")
+		(pts
+			(xy 170.25 105.5) (xy 170.25 108.75)
+		)
+		(height 8.25)
+		(gr_text "3.2500 mm"
+			(at 160.85 107.125 90)
+			(layer "Edge.Cuts")
+			(effects
+				(font
+					(size 1 1)
+					(thickness 0.15)
+				)
+			)
+		)
+		(format
+			(prefix "")
+			(suffix "")
+			(units 3)
+			(units_format 1)
+			(precision 4)
+		)
+		(style
+			(thickness 0.05)
+			(arrow_length 1.27)
+			(text_position_mode 0)
+			(extension_height 0.58642)
+			(extension_offset 0.5) keep_text_aligned)
+	)
+	(dimension
+		(type aligned)
+		(layer "Edge.Cuts")
+		(pts
+			(xy 170.25 105.5) (xy 170.25 90.5)
+		)
+		(height -11)
+		(gr_text "15.0000 mm"
+			(at 158.1 98 90)
+			(layer "Edge.Cuts")
+			(effects
+				(font
+					(size 1 1)
+					(thickness 0.15)
+				)
+			)
+		)
+		(format
+			(prefix "")
+			(suffix "")
+			(units 3)
+			(units_format 1)
+			(precision 4)
+		)
+		(style
+			(thickness 0.05)
+			(arrow_length 1.27)
+			(text_position_mode 0)
+			(extension_height 0.58642)
+			(extension_offset 0.5) keep_text_aligned)
+	)
 	(segment
